File: 20201114_volume.kicad_pcb (KiCad board)
At the start: 2 copper layers, 110 x 50 mm, 146 parts, among them J101 POWER, J102 POWER_SW_DETECT, J103 8P8C_Shielded, J104 AudiotoMCU, J105 MCUtoAudio, J106 ENC, J107 SWD, J108 LEDtoMCU, J109 MCUtoLED, J110 Mute, J111 Mute, J112 SW, J301 POWER, J302 IN, J303 IN, Q101 2N7002K, Q102 2N7002K, Q201 2N7002K, Q202 2N7002K, Q203 2N7002K, Q204 IRLML2246TRPbF, Q205 2N7002K, Q206 2N7002K, Q207 2N7002K, Q208 IRLML2246TRPbF, Q209 2N7002K, Q210 2N7002K, Q211 2N7002K, Q212 IRLML2246TRPbF, Q213 2N7002K, Q214 2N7002K, Q301 TTC004B, Q302 TTA004B, Q303 TTC004B, Q304 TTA004B, Q305 TTC004B, Q306 TTA004B, Q307 TTC004B, Q308 TTA004B, Q309 TTC004B, Q310 TTA004B, Q311 TTC004B, Q312 TTA004B, Q313 [mu]PA2753GR, Q314 [mu]PA2753GR, U101 TLP785, U102 NJW1933-T, U103 NJU7223FDL1-33, U104 STM32F042K6Tx, U301 OPAMP, U302 LM1972, U303 OPAMP, U304 TLP4227G, U305 TLP591B, U306 TLP4227G, U307 TLP591B

Commit message: v1.0
Parts:
- removed J112: SW, Connector_JST:JST_XH_B3B-XH-A_1x03_P2.50mm_Vertical
- removed Q301, Q303: TTC004B, Package_TO_SOT_THT:TO-126-3_Vertical
- removed Q302, Q304: TTA004B, Package_TO_SOT_THT:TO-126-3_Vertical
- removed R101: 1k, Resistor_SMD:R_0603_1608Metric_Pad1.05x0.95mm_HandSolder
- removed R303: 0, Resistor_THT:R_Axial_DIN0204_L3.6mm_D1.6mm_P5.08mm_Horizontal
- removed R304, R305: 1.2k, Resistor_THT:R_Axial_DIN0204_L3.6mm_D1.6mm_P5.08mm_Horizontal
- removed R306, R307: 4.7, Resistor_THT:R_Axial_DIN0204_L3.6mm_D1.6mm_P5.08mm_Horizontal
- removed U301: OPAMP, Package_DIP:DIP-8_W7.62mm_Socket
- added C109: NC 47u, Capacitor_THT:CP_Radial_D6.3mm_P2.50mm, F.Cu at (63.3, 107.2)
- added G***: LOGO, kele:kele2, F.Cu at (68.4, 124.3)
- added G***: LOGO, kele:kele2, B.Cu at (106.5, 73.5)
- added H101: mounting_hole, fues-mounting_hole:M3-drillHole_6mm_nosilk_nopad, F.Cu at (53.5, 134.5)
- added H102: mounting_hole, fues-mounting_hole:M3-drillHole_6mm_nosilk_nopad, F.Cu at (106.5, 124.5)
- added H103: mounting_hole, fues-mounting_hole:M3-drillHole_6mm_nosilk_nopad, F.Cu at (53.5, 105.5)
- added H104: mounting_hole, fues-mounting_hole:M3-drillHole_6mm_nosilk_nopad, F.Cu at (106.5, 105.5)
- added H301: mounting_hole, fues-mounting_hole:M3-drillHole_6mm_nosilk_nopad, F.Cu at (118.5, 53.5)
- added H302: mounting_hole, fues-mounting_hole:M3-drillHole_6mm_nosilk_nopad, F.Cu at (118.5, 96.5)
- added H303: mounting_hole, fues-mounting_hole:M3-drillHole_6mm_nosilk_nopad, F.Cu at (53.5, 53.5)
- added H304: mounting_hole, fues-mounting_hole:M3-drillHole_6mm_nosilk_nopad, F.Cu at (53.5, 96.5)
- added TP101: TestPoint, TestPoint:TestPoint_THTPad_D1.0mm_Drill0.5mm, F.Cu at (77.9, 128.2)
- C101, C102, C104, C105, C108, L101, Q101, Q102, R102, R103, R104, R105, R108, U102: moved to B.Cu
- C302: value 0.1u -> NC
- C303, C307, C308, C309: moved to F.Cu
- H201, H202: footprint MountingHole:MountingHole_3.2mm_M3_DIN965 -> fues-mounting_hole:M3-drillHole_6mm_nosilk_nopad
- J102, J110, J111: footprint Connector_JST:JST_XH_B2B-XH-A_1x02_P2.50mm_Vertical -> fues-connect:JST_ZH_B2B-ZR_1x02_P1.50mm_Vertical
- J103: footprint Connector_RJ:RJ45_Amphenol_RJHSE5380 -> fues-connect:7810-8P8C
- J104, J105: footprint Connector_JST:JST_XH_B4B-XH-A_1x04_P2.50mm_Vertical -> fues-connect:JST_ZH_B4B-ZR_1x04_P1.50mm_Vertical
- J106: footprint Connector_JST:JST_XH_B3B-XH-A_1x03_P2.50mm_Vertical -> fues-connect:JST_ZH_B6B-ZR_1x06_P1.50mm_Vertical
- J107: footprint Connector_PinHeader_1.27mm:PinHeader_1x05_P1.27mm_Vertical -> Connector_PinSocket_1.27mm:PinSocket_1x05_P1.27mm_Vertical
- R301, R302: value 10k -> 1k; footprint Resistor_SMD:R_0603_1608Metric_Pad1.05x0.95mm_HandSolder -> Resistor_THT:R_Axial_DIN0207_L6.3mm_D2.5mm_P10.16mm_Horizontal; moved to F.Cu
- R320, R322: value 30 -> 1k; footprint Capacitor_SMD:C_0603_1608Metric_Pad1.05x0.95mm_HandSolder -> Resistor_SMD:R_0603_1608Metric_Pad1.05x0.95mm_HandSolder
- R321, R323: value 30 -> 500; footprint Capacitor_SMD:C_0603_1608Metric_Pad1.05x0.95mm_HandSolder -> Resistor_SMD:R_0603_1608Metric_Pad1.05x0.95mm_HandSolder
- R324, R325, R326, R327: value 30 -> 220; footprint Capacitor_SMD:C_0603_1608Metric_Pad1.05x0.95mm_HandSolder -> Resistor_SMD:R_0603_1608Metric_Pad1.05x0.95mm_HandSolder
- moved Q101 135.6 mm to (63.2, 122.2), turned to 90 degrees
- moved R104 135.3 mm to (63.2, 124.8)
- moved R320 132.3 mm to (95.7, 96.4), turned to 90 degrees
- moved R103 131.3 mm to (62.5, 116.1), turned to 180 degrees
- moved R102 128.9 mm to (60.4, 122.3), turned to 90 degrees
- moved R108 128.2 mm to (68.4, 130.9), turned to 90 degrees
- moved R105 127.5 mm to (68.4, 121.8)
- moved R324 124.1 mm to (91.9, 96.4), turned to 270 degrees
- moved C107 123.0 mm to (99.0, 126.0), turned to 90 degrees
- moved C108 118.9 mm to (81.8, 121.2), turned to 270 degrees
- moved R325 118.4 mm to (91.9, 88.7), turned to 270 degrees
- moved J103 117.0 mm to (55.0, 120.0), turned to 270 degrees
- moved R322 115.5 mm to (63.3, 96.4), turned to 90 degrees
- moved R321 115.2 mm to (95.7, 91.3), turned to 270 degrees
- moved C101 112.4 mm to (95.0, 109.1), turned to 180 degrees
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Connections:
- net Net-(D102-Pad1) renamed /5Vsw
- C302 pad 1: Net-(C302-Pad1) -> VDDA
- C302 pad 2: VSSA -> GNDA
- C306 pad 1: Net-(C306-Pad1) -> GNDA
- C306 pad 2: Net-(C306-Pad2) -> VSSA
- J102 pad 2: Net-(J102-Pad2) -> /power_sw
- Q314 pad 5: Net-(Q314-Pad5) -> /Audio/fb2
- Q314 pad 6: Net-(Q314-Pad5) -> /Audio/fb2
- Q314 pad 7: /Audio/fb2 -> Net-(Q314-Pad7)
- Q314 pad 8: /Audio/fb2 -> Net-(Q314-Pad7)
- R301 pad 2: Net-(C302-Pad1) -> GNDA
- R302 pad 1: Net-(C302-Pad1) -> GNDA
- R329 pad 2: Net-(Q314-Pad5) -> Net-(Q314-Pad7)
- R331 pad 2: Net-(Q314-Pad5) -> Net-(Q314-Pad7)
- U104 pad 26: /BTN_1 -> /vol_dat
- U104 pad 27: /BTN_2 -> /vol_load
- U104 pad 28: /BTN_3 -> /vol_clk
- U104 pad 29: /vol_dat -> /BTN_1
- U104 pad 30: /vol_load -> /BTN_2
- U104 pad 31: /vol_clk -> /BTN_3
- U303 pad 1: Net-(C312-Pad1) -> Net-(C313-Pad1)
- U303 pad 2: Net-(C312-Pad2) -> Net-(C313-Pad2)
- U303 pad 3: /Audio/volout1 -> /Audio/volout2
- U303 pad 5: /Audio/volout2 -> /Audio/volout1
- U303 pad 6: Net-(C313-Pad2) -> Net-(C312-Pad2)
- U303 pad 7: Net-(C313-Pad1) -> Net-(C312-Pad1)
Routing:
- net GNDA: track 98.5 -> 310.1 mm, vias 0 -> 18
- net GND: track 0.00 -> 208.8 mm, vias 0 -> 6
- net +5V: track 0.00 -> 167.0 mm, vias 0 -> 7
- net VDDA: track 46.8 -> 206.7 mm, vias 0 -> 2
- net VSSA: track 24.8 -> 178.6 mm, vias 0 -> 2
- net /Audio/mute-: track 0.00 -> 74.3 mm
- net +3V3: track 0.00 -> 62.7 mm, vias 0 -> 4
- net Net-(Q314-Pad1): track 0.00 -> 62.5 mm
- net Net-(Q313-Pad1): track 0.00 -> 61.8 mm
- net Net-(Q314-Pad2): track 0.00 -> 61.2 mm, vias 0 -> 1
- net Net-(Q313-Pad2): track 0.00 -> 61.2 mm, vias 0 -> 1
- net /Audio/mute+: track 0.00 -> 60.5 mm, vias 0 -> 1
- net /Audio/dat: track 0.00 -> 52.5 mm, vias 0 -> 3
- net /display/K_G: track 1.62 -> 51.6 mm, vias 0 -> 1
- net /display/A_COM3: track 1.62 -> 50.5 mm, vias 0 -> 1
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- added copper zone on B.Cu, net +5V
- added copper zone on F.Cu, net +5V
- added copper zone on B.Cu, net GND
- added copper zone on F.Cu, net GND
- added copper zone on B.Cu, net GNDA
- added copper zone on F.Cu, net GNDA
Other:
- board size 110 x 50 mm -> 96 x 88 mm
- board text added: "audio volume PCB:Audio ver 1.0 2021/07/24 kamibushiele.net"
- board text added: "audio volume PCB:MCU ver 1.0 2021/07/24 kamibushiele.net"
- board text added: "kamibushiele.net"
- board text added: "ver 1.0 2021/ 07/24"
